File: kicad/storm_distance_meter.kicad_pcb (KiCad board)
At the start: 2 copper layers, 36 x 110 mm, 50 parts, among them J1 Terminal RM3.5, Q1 BC546, Q2 BC556, Q3 BC546, Q4 BC546, SW1 6mm, SW2 6mm, SW3 6mm, SW4 7x7mm, U1 NE555P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

Commit message: Updated PCB, manuals
Other:
- board text added: "v2"
- board text removed: "v1"
